Commit message: change laser position, no colide anymore

File: p3dx_description/urdf/pioneer3dx.xacro (robot description, xacro)
@@ -218,5 +218,6 @@
 	<joint name="lms100_joint" type="fixed">
 		<axis xyz="0 1 0" />
-		<origin xyz="0.12 0 0.26" rpy="0 0 0" />
+		<!--origin xyz="0.12 0 0.26" rpy="0 0 0" /-->
+		<origin xyz="0.12 0 0.185" rpy="0 0 0" />
 		<parent link="base_link" />
 		<child link="lms100" />
